File: 01_eagle/omcPendelautomatik_tapein.brd (EAGLE design)
At the start: 44.5 x 69.8 mm, 71 parts, among them IC1 PIC12F675, IC2 7805, IC3 L5970D, K1 NA-5V, T1 BSS138, T2 BSS138, X1 RT034 Typ 086, X2 2X3

Commit message: omcPendelautomatik -> added label with name and version
Routing:
- added copper zone on layer 16, net N$31
Other:
- board text added: "OMC Adorf"
- board text added: "V1.0, 04/2019"
- board text added: "omcPendelautomatik"
Changed lines of the file:
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@@
 <text x="27.94" y="67.6275" size="1.4224" layer="1" font="vector" ratio="15">+TIV-</text>
 <text x="27.94" y="67.6275" size="1.4224" layer="25" font="vector" ratio="15">+TIV-</text>
+<text x="10.16" y="67.31" size="1.016" layer="16" font="vector" ratio="15" rot="MR180">omcPendelautomatik</text>
+<text x="10.16" y="66.04" size="1.016" layer="16" font="vector" ratio="15" rot="MR180">OMC Adorf</text>
+<text x="10.16" y="64.77" size="1.016" layer="16" font="vector" ratio="15" rot="MR180">V1.0, 04/2019</text>
 </plain>
 <attributes>
@@
 <vertex x="27.305" y="20.955"/>
 </polygon>
+<via x="22.225" y="60.96" extent="1-16" drill="0.4" diameter="0.8128" shape="octagon"/>
 </signal>
 <signal name="VOUT">
@@
 </polygon>
 </signal>
+<signal name="N$31">
+<polygon width="0.4064" layer="16" pour="cutout">
+<vertex x="10.16" y="67.31"/>
+<vertex x="10.16" y="63.5"/>
+<vertex x="21.59" y="63.5"/>
+<vertex x="21.59" y="66.04"/>
+<vertex x="26.035" y="66.04"/>
+<vertex x="26.035" y="67.31"/>
+</polygon>
+</signal>
