File: 01_eagle/omcPendelautomatik.sch (EAGLE design)
At the start: 57 parts, among them IC1 L5970D, IC2 7805, IC3 TLC555, K1 NA-5V, X1 RT034 Typ 086

Commit message: omcPendelautomatik.sch -> intermediate commit -> changed from '555' timing normal to 'uC'
Parts:
- added B1: JTP1138/4.3, omcSwitch:JTP1138-4.3MM
- added C20: 100n, omcCapacitor:X7R-100000P-1206
- added H1, H2, H3, H4: MOUNT-PAD-ROUND3.2, holes:MOUNT-PAD-ROUND3.2
- added LED2: Red, omcOpto:LEDMONO-RED-KP3216
- added R19: 39K, omcResistor:RC1206-39000
- added R20: 10K, omcResistor:RC1206-10000
- added R21: 1K, omcResistor:RC1206-1000
- added T1, T2: BSS138, omcTransistor:BSS138
- added X5: PH2X3, omcConnector:PH2X3-P1.27
- C11: value 100n -> 100n/50V
- C12: value 100n -> 2n2; device omcCapacitor:X7R-100000P-1206 -> omcCapacitor:NP0-2200P-1206
- C13: value 100µ -> 100n/50V; device omcCapacitor:X5R-100000000P-1210 -> omcCapacitor:X7R-100000P-1206
- C16, C17, C18, C19: value 10n -> 10n/50V
- D2, D3, D4, D5: value 1N4148 -> PMEG4010; device omcDiode:1N4148LL -> omcDiode:PMEGXX10-40VBEA
- IC3: value TLC555 -> PIC12F675; device omcReferences:TLC555ID -> omcPIC:PIC12F675SN
- R10: value 10K -> 1K; device omcResistor:RC1206-10000 -> omcResistor:RC1206-1000
- R11: value 100K -> 1K; device omcResistor:M44-100000W -> omcResistor:RC1206-1000
- R13: value 0R -> 10K; device omcResistor:RC1206-0.0 -> omcResistor:RC1206-10000
- R16: value 7K5 -> 56K; device omcResistor:RC1206-7500 -> omcResistor:RC1206-56000
- R17: value 360R -> 10K; device omcResistor:RC1206-360 -> omcResistor:RC1206-10000
- R18: value 33K -> 10K; device omcResistor:RC1206-33000 -> omcResistor:M44-10000W
- R8: value 10K -> 56K; device omcResistor:RC1206-10000 -> omcResistor:RC1206-56000
- R9: value 10K -> 22K; device omcResistor:RC1206-10000 -> omcResistor:RC1206-22000
Connections:
- removed net VR: R16.2
- new net ICSPCLK: IC3.1, R11.1, X5G$5.P$1
- new net ICSPDAT: IC3.0, R10.1, X5G$4.P$1
- new net I_VCC: C12.2, OPA1G$1.OUT, R10.2, R19.2
- new net N$27: IC3.2, LED2.C, R21.2
- new net N$28: B1.P$3, B1.P$4, R21.1
- new net REGON: IC1.INH, T2.D
- new net RLON: D5.A, K1G$1.1, LED1.C, T1.D
- net +5V: now also C20.2, D3.A, D4.A, LED2.A, R18.A; no longer C11.1, IC3.VCC+, R10.2, R9.2
- net GND: now also B1.P$1, B1.P$2, C20.1, H1.MOUNT, H2.MOUNT, H3.MOUNT, H4.MOUNT, IC3.VSS, R16.1, R18.E, R20.1, R8.1, T1.S, T2.S, X5G$3.P$1; no longer C12.2, IC3.GND, R17.1
- net N$10: now also IC3.!MCLR!, R9.1, X5G$1.P$1; no longer D3.C, D4.A, IC3.!TRI, IC3.TRE, R11.E, R13.2
- net N$11: now also D4.C, R9.2; no longer D3.A, IC3.DIS, R10.1, R8.2
- net N$12: now also IC3.5, R13.2; no longer IC3.!RES, R9.1
- net N$13: now also R16.2, R17.1, T2.G; no longer D5.A, IC3.OUT, K1G$1.1, LED1.C
- net N$14: now also IC3.4, R17.2; no longer C13.1, R11.A, R11.S, R13.1
- net N$19: now also C11.1, R11.2, R18.S; no longer OPA1G$1.OUT, R18.2
- net N$20: now also C12.1, OPA1G$1.-IN, R19.1, R20.2; no longer OPA1G$1.+IN, R16.1, R17.2, R18.1
- net N$5: now also R13.1, R8.2, T1.G; no longer D4.C, R8.1
- net N$7: now also C13.1, D3.C, IC3.VDD, X5G$2.P$1; no longer C12.1, IC3.CON
- net V_ISNS: now also OPA1G$1.+IN; no longer OPA1G$1.-IN
Other:
- note added: "ICSP Interface"
- note added: "V_ISNS [V] = I_VCC [A]"
- note added: "over-current reset button"
- note removed: "VTH=0.15V VTL=0.20V"
- note removed: "http://sim.okawa-denshi.jp/en/compkeisan.htm"
- note removed: "https://www.elektronik-kompendium.de/sites/slt/0310131.htm"
- moved on the sheet: C11, C12, C13, C3, C6, D3, D4, D5, D6, D7, D8, D9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

Commit message: omcPendelautomatik.sch -> initial draft schematic finished
Parts:
- removed X5: PH2X3, omcConnector:PH2X3-P1.27
- added X2: PH2X3, omcConnector:PH2X3-SMD1.27
- C1: value 10µ/35V -> 10n/50V; device omcCapacitor:X7R-10000000P-1210 -> omcCapacitor:X7R-10000P-1206
- C10: value 2µ2/50V -> 100n/50V; device omcCapacitor:X7R-2200000P-1206 -> omcCapacitor:X7R-100000P-1206
- C12: value 2n2 -> 2µ2/50V; device omcCapacitor:NP0-2200P-1206 -> omcCapacitor:X7R-2200000P-1206
- C13: value 100n/50V -> 220p/50V; device omcCapacitor:X7R-100000P-1206 -> omcCapacitor:NP0-220P-1206
- C14: value 150µ/35V -> 22n/50V; device omcCapacitor:AEC-150U-35V-F -> omcCapacitor:X7R-22000P-1206
- C15: value 150µ/35V -> 100n; device omcCapacitor:AEC-150U-35V-F -> omcCapacitor:X7R-100000P-1206
- C16: value 10n/50V -> 2n2; device omcCapacitor:X7R-10000P-1206 -> omcCapacitor:NP0-2200P-1206
- C17, C18: value 10n/50V -> 100n/50V; device omcCapacitor:X7R-10000P-1206 -> omcCapacitor:X7R-100000P-1206
- C19: value 10n/50V -> 47µ/16V; device omcCapacitor:X7R-10000P-1206 -> omcCapacitor:X5R-47000000P-1210
- C2, C5: value 100n/50V -> 10n/50V; device omcCapacitor:X7R-100000P-1206 -> omcCapacitor:X7R-10000P-1206
- C20: value 100n -> 47µ/16V; device omcCapacitor:X7R-100000P-1206 -> omcCapacitor:X5R-47000000P-1210
- C3: value 22n/50V -> 100n/50V; device omcCapacitor:X7R-22000P-1206 -> omcCapacitor:X7R-100000P-1206
- C4: value 47µ/16V -> 10n/50V; device omcCapacitor:X5R-47000000P-1210 -> omcCapacitor:X7R-10000P-1206
- C6: value 220p/50V -> 150µ/35V; device omcCapacitor:NP0-220P-1206 -> omcCapacitor:AEC-150U-35V-F
- C7: value 100n/50V -> 2µ2/50V; device omcCapacitor:X7R-100000P-1206 -> omcCapacitor:X7R-2200000P-1206
- C8: value 2µ2/50V -> 150µ/35V; device omcCapacitor:X7R-2200000P-1206 -> omcCapacitor:AEC-150U-35V-F
- C9: value 47µ/16V -> 10µ/35V; device omcCapacitor:X5R-47000000P-1210 -> omcCapacitor:X7R-10000000P-1210
- D1: value MBRS240 -> PMEG4010; device omcDiode:MBRS240 -> omcDiode:PMEGXX10-40VBEA
- D4: value PMEG4010 -> MBRS240; device omcDiode:PMEGXX10-40VBEA -> omcDiode:MBRS240
- IC1: value L5970D -> PIC12F675; device omcPwrSupply:L5970D -> omcPIC:PIC12F675SN
- IC3: value PIC12F675 -> L5970D; device omcPIC:PIC12F675SN -> omcPwrSupply:L5970D
- LED1: value Yellow -> Red; device omcOpto:LEDMONO-YELLOW-KP3216 -> omcOpto:LEDMONO-RED-KP3216
- LED2: value Red -> Yellow; device omcOpto:LEDMONO-RED-KP3216 -> omcOpto:LEDMONO-YELLOW-KP3216
- R1: value 3K3 -> 22K; device omcResistor:RC1206-3300 -> omcResistor:RC1206-22000
- R11: value 1K -> 39K; device omcResistor:RC1206-1000 -> omcResistor:RC1206-39000
- R12: value 1K -> 10K; device omcResistor:RC1206-1000 -> omcResistor:M44-10000W
- R13: value 10K -> 1K; device omcResistor:RC1206-10000 -> omcResistor:RC1206-1000
- R14: value 50K -> 1R; device omcResistor:M44-50000W -> omcResistor:RC1206-1.0
- R15: value 0R -> 1R; device omcResistor:RC1206-0.0 -> omcResistor:RC1206-1.0
- R16: value 56K -> 200R; device omcResistor:RC1206-56000 -> omcResistor:RC1206-200
- R17: value 10K -> 0R; device omcResistor:RC1206-10000 -> omcResistor:RC1206-0.0
- R18: value 10K -> 47K; device omcResistor:M44-10000W -> omcResistor:RC1206-47000
- R19: value 39K -> 3K3; device omcResistor:RC1206-39000 -> omcResistor:RC1206-3300
- R2: value 47K -> 10K; device omcResistor:RC1206-47000 -> omcResistor:RC1206-10000
- R20: value 10K -> 50K; device omcResistor:RC1206-10000 -> omcResistor:M44-50000W
- R21: value 1K -> 4K7; device omcResistor:RC1206-1000 -> omcResistor:RC1206-4700
- R3: value 4K7 -> 56K; device omcResistor:RC1206-4700 -> omcResistor:RC1206-56000
- R4: value 4K7 -> 1K; device omcResistor:RC1206-4700 -> omcResistor:RC1206-1000
- R5: value 1R -> 1K; device omcResistor:RC1206-1.0 -> omcResistor:RC1206-1000
- R6: value 1R -> 10K; device omcResistor:RC1206-1.0 -> omcResistor:RC1206-10000
- R7: value 200R -> 56K; device omcResistor:RC1206-200 -> omcResistor:RC1206-56000
- R8: value 56K -> 4K7; device omcResistor:RC1206-56000 -> omcResistor:RC1206-4700
- R9: value 22K -> 10K; device omcResistor:RC1206-22000 -> omcResistor:RC1206-10000
Connections:
- net +5V: now also C10.1, C12.1, C15.2, D1.A, D2.A, LED1.A, R12.A, R13.2; no longer C20.2, C5.1, C8.1, D3.A, D4.A, LED2.A, R12.2, R18.A
- net GND: now also C12.2, C13.1, C15.1, C17.2, C18.2, C19.2, C2.1, C20.2, C3.2, C6.-, C8.-, D4.A, IC1.VSS, IC3.GND, R12.E, R19.1, R3.1, R9.1, X2G$3.P$1; no longer C13.2, C14.-, C15.-, C16.2, C17.1, C2.2, C20.1, C4.2, C5.2, C6.1, C8.2, D1.A, IC1.GND, IC3.VSS, R1.1, R18.E, R20.1, R4.1, X5G$3.P$1
- net ICSPCLK: now also IC1.1, R5.1, X2G$5.P$1; no longer IC3.1, R11.1, X5G$5.P$1
- net ICSPDAT: now also IC1.0, R4.1, X2G$4.P$1; no longer IC3.0, R10.1, X5G$4.P$1
- net I_VCC: now also C16.2, R11.2, R4.2; no longer C12.2, R10.2, R19.2
- net N$1: now also D4.C, IC3.OUT; no longer D1.C, IC1.OUT
- net N$10: now also IC1.!MCLR!, R1.1, X2G$1.P$1; no longer IC3.!MCLR!, R9.1, X5G$1.P$1
- net N$11: now also D2.C, R1.2; no longer D4.C, R9.2
- net N$12: now also IC1.5, R2.2; no longer IC3.5, R13.2
- net N$13: now also R6.1, R7.2; no longer R16.2, R17.1
- net N$14: now also IC1.4, R6.2; no longer IC3.4, R17.2
- net N$15: now also LED2.A, R13.1; no longer LED1.A, R12.1
- net N$16: now also R17.1, R18.2; no longer R15.1, R2.2
- net N$17: now also C1.1, C4.1; no longer C16.1, C18.1
- net N$19: now also C17.1, R12.S, R5.2; no longer C11.1, R11.2, R18.S
- net N$2: now also R20.A, R20.S, R21.2; no longer R14.A, R14.S, R3.2
- net N$20: now also C16.1, R11.1, R9.2; no longer C12.1, R19.1, R20.2
- net N$21: now also D7.A; no longer D9.A
- net N$23: now also C2.2, C5.2; no longer C17.2, C19.2
- net N$25: now also D9.A; no longer D7.A
- net N$27: now also IC1.2, LED1.C, R10.2; no longer IC3.2, LED2.C, R21.2
- net N$28: now also R10.1; no longer R21.1
- net N$3: now also C13.2, C14.1, IC3.COMP; no longer C3.1, C6.2, IC1.COMP
- net N$4: now also C14.2, R8.2; no longer C3.2, R4.2
- net N$5: now also R2.1, R3.2; no longer R13.1, R8.2
- net N$6: now also C11.1, C4.2, C5.1, C6.+, C7.1, C8.+, C9.1, D3.C, IC3.VCC; no longer C1.1, C10.1, C14.+, C15.+, C18.2, C19.1, C2.1, D2.C, IC1.VCC
- net N$7: now also C3.1, D1.C, IC1.VDD, X2G$2.P$1; no longer C13.1, D3.C, IC3.VDD, X5G$2.P$1
- net N$9: now also IC3.FB, R18.1, R19.2, R21.1; no longer IC1.FB, R1.2, R2.1, R3.1
- net REGON: now also IC3.INH; no longer IC1.INH
- net RLON: now also LED2.C; no longer LED1.C
- net VCC: now also R14.2, R17.2, R20.E; no longer R14.E, R5.2, R6.2
- net VOUT: now also C18.1, C19.1, C20.1, D3.A, R14.1, R15.1; no longer C4.1, C7.1, C9.1, D2.A, R5.1, R6.1
- net V_ISNS: now also R16.2; no longer R7.2
Other:
- moved on the sheet: C1, C10, C11, C12, C13, C16, C17, C18, C19, C2, C20, C3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
